Commit message: Update smr1000_description.urdf
Add Lidar merged link

File: urdf/smr1000_description.urdf (robot description, URDF)
Before this commit: robot smr1000_description, 26 links, 25 joints
Links:
- added link lidar_merged_link
Joints:
- added joint base_link_to_lidar_merged_link: type fixed, parent base_link, child lidar_merged_link, origin xyz=0.0 0.0 0.1 rpy=0 0 0

Commit message: Update smr1000_description.urdf

File: urdf/smr1000_description.urdf (robot description, URDF)
Before this commit: robot smr1000_description, 27 links, 26 joints
Joints:
- joint base_link_to_lidar_merged_link: origin xyz=0.0 0.0 0.1 rpy=0 0 0 -> xyz=0.0 0.0 0.1198 rpy=0 0 0

Commit message: Update smr1000_description.urdf

File: urdf/smr1000_description.urdf (robot description, URDF)
Before this commit: robot smr1000_description, 27 links, 26 joints
Links:
- added link depthcam_front_left_view_link, mass 0.001
Joints:
- added joint depthcam_front_left_view_joint: type fixed, parent depth_cam_front_left_mount_point_link, child depthcam_front_left_view_link, origin xyz=0.0 0.0 0.0 rpy=-1.5708 0.0 -1.5708
- added joint depthcam_front_right_view_joint: type fixed, parent depth_cam_front_right_mount_point_link, child depthcam_front_right_view_link, origin xyz=0.0 0.0 0.0 rpy=-1.5708 0.0 -1.5708

Commit message: Update smr1000_description.urdf

File: urdf/smr1000_description.urdf (robot description, URDF)
Before this commit: robot smr1000_description, 28 links, 28 joints
Links:
- added link depthcam_front_right_view_link, mass 0.001

Commit message: Update smr1000_description.urdf

File: urdf/smr1000_description.urdf (robot description, URDF)
Before this commit: robot smr1000_description, 29 links, 28 joints
Links:
- removed link depth_cam_front_left_mount_point_link
- removed link depth_cam_front_right_mount_point_link
- added link depthcam_front_left_link, mass 0.0375455045895058; collision mesh filename=package://smr1000_description/meshes/depthcam_front_left_li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; visual mesh filename=package://smr1000_description/meshes/depthcam_front_left_li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
- added link depthcam_front_right_link, mass 0.0375455004175735; collision mesh filename=package://smr1000_description/meshes/depthcam_front_right_l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; visual mesh filename=package://smr1000_description/meshes/depthcam_front_right_l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
Joints:
- joint depth_cam_front_left_mount_point_joint: child depth_cam_front_left_mount_point_link -> depthcam_front_left_link
- joint depth_cam_front_right_mount_point_joint: child depth_cam_front_right_mount_point_link -> depthcam_front_right_link
- joint depthcam_front_left_view_joint: parent depth_cam_front_left_mount_point_link -> depthcam_front_left_link
- joint depthcam_front_right_view_joint: parent depth_cam_front_right_mount_point_link -> depthcam_front_right_link
